File: Magi.kicad_pcb (KiCad board)
At the start: 6 copper layers, 122 x 85 mm, 428 parts, among them J1 Micro_SD_Card_Det2, J10 Conn_02x02_Odd_Even, J11 USB_C_Receptacle, J12 USB_C_Receptacle, J2 Bus_M.2_Socket_M, J3 Micro_SD_Card_Det2, J4 Bus_M.2_Socket_M, J5 Micro_SD_Card_Det2, J6 Bus_M.2_Socket_M, J7 RJ45_LED_Shielded, J8 USB_C_Receptacle, J9 Conn_02x04, Q1 DMN32D2LFB4, Q2 DMN32D2LFB4, Q3 DMN32D2LFB4, Q4 DMN32D2LFB4, SW1 SW_Push, U1 TPS56339DDC, U10 TPS56339DDC, U11 AP2151W, U12 74AUP1G125, U13 RTL8367S-CG, U14 TPD4EUSB30, U15 TPD4EUSB30, U16 USB2514B, U17 CH390H, U18 STM32G0B1VETx, U19 TPD4EUSB30, U2 TPS56339DDC, U20 TPS259470A, U21 TPS259470A, U22 TPS259470A, U23 TPS259470A, U24 TPS259470A, U25 TPS259470A, U26 TPS56339DDC, U27 TPS259470A, U28 TPS56339DDC, U29 TVS2200DRV, U3 AP2151W, U30 TPD6S300A, U31 FUSB340TMX, U32 TPD4EUSB30, U33 TS3USB221, U34 TPD4EUSB30, U35 AP2151W, U36 AP2151W, U37 TS3USB221, U38 TPD6S300A, U39 TVS2200DRV, U4 74AUP1G125, U40 HD3SS460, U41 TPD4EUSB30, U42 AP2151W, U43 TPD4EUSB30, U44 AP2151W, U5 TPS56339DDC, U6 TPS56339DDC, U7 AP2151W, U8 74AUP1G125, U9 TPS56339DDC, Y1 25MHz, Y2 25MHz, Y3 24MHz, Y4 32.768kHz

Commit message: Magi v2.1
Parts:
- removed R63: 2.49K, Resistor_SMD:R_0402_1005Metric
- removed kibuzzard-6A5B157A: G***, kibuzzard-6A5B157A
- added C190: 100n, Capacitor_SMD:C_0402_1005Metric, F.Cu at (151.1, 53.6)
- added C191: 100n, Capacitor_SMD:C_0402_1005Metric, F.Cu at (149.5, 58.8)
- added R116: 5.1k, Resistor_SMD:R_0402_1005Metric, F.Cu at (154.0, 57.7)
- added R117: 5.1k, Resistor_SMD:R_0402_1005Metric, F.Cu at (154.0, 54.9)
- added TP12: TestPoint, TestPoint:TestPoint_Pad_D1.5mm, B.Cu at (153.0, 119.0)
- added TP13: TestPoint, TestPoint:TestPoint_Pad_D1.5mm, B.Cu at (164.5, 66.5)
- added TP16: TestPoint, TestPoint:TestPoint_Pad_D1.5mm, B.Cu at (165.5, 105.0)
- added U45: ATECC608B-MAHCZ, Package_DFN_QFN:DFN-8-1EP_3x2mm_P0.5mm_EP1.3x1.5mm, F.Cu at (151.2, 60.5)
- added U46: CAT25512HU5I-GT3, Magi:DFN-8-1EP_3x2mm_P0.5mm_EP0.9x1.4mm, F.Cu at (151.2, 56.2)
- added kibuzzard-6AC565B3: G***, kibuzzard-6AC565B3, F.Cu at (158.8, 105.7)
- D10, D7, D8, D9: value WS2812B -> WS2812C; footprint Magi:LED-SMD_4P-L4.0-W1.7-R -> Magi:LED-SMD_4P-L4.0-W1.7_DCS
- moved TP2 3.00 mm to (199.5, 101.0), turned to 0 degrees
- moved J10 0.50 mm to (210.5, 55.5)
- moved R57 0.30 mm to (153.5, 56.3)
- moved R58 0.30 mm to (154.5, 56.3)
- turned D10 to 0 degrees
- turned D7 to 180 degrees
- turned D8 to 0 degrees
- turned D9 to 0 degrees
- renumbered TP12 to TP14, TP13 to TP15
Connections:
- J9 pad 5: GND -> /Controller/PD11_SPI3_INT
- Module1 pad 24: /Controller/PF1 -> unconnected-(Module1A-GPIO26-Pad24)
- Module1 pad 93: /Controller/PC13 -> /Controller/PC12
- Module2 pad 24: /Controller/PB0 -> unconnected-(Module2A-GPIO26-Pad24)
- Module3 pad 24: /Controller/PD11 -> unconnected-(Module3A-GPIO26-Pad24)
- R113 pad 1: /Controller/MCU_BUTTON -> /Controller/PB0_MCU_BUTTON
- R54 pad 1: Net-(U16-RESET_N) -> /Controller/PF1
- SW1 pad 1: /Controller/MCU_BUTTON -> /Controller/PB0_MCU_BUTTON
- U16 pad 26: Net-(U16-RESET_N) -> /Controller/PF1
- U18 pad 35: /Controller/PB0 -> /Controller/PB0_MCU_BUTTON
- U18 pad 58: unconnected-(U18-PC7-Pad58) -> /Controller/PC7
- U18 pad 62: /Controller/PD11 -> /Controller/PD11_SPI3_INT
- U18 pad 84: /Controller/MCU_BUTTON -> /Controller/PD6_USART2_RX
- U38 pad 15: /Controller/PF9_USART6_TX -> /Controller/PD6_USART2_RX
- U40 pad 3: /Controller/PC12 -> /Controller/PC13
Routing:
- net /Controller/PC7: track 0.00 -> 87.3 mm, vias 0 -> 3
- net /Controller/MCU_BUTTON: track 86.2 -> 0.00 mm, vias 2 -> 0
- net /Controller/PB0_MCU_BUTTON: track 0.00 -> 71.9 mm, vias 0 -> 2
- net /Controller/PD11: track 57.7 -> 0.00 mm, vias 2 -> 0
- net /Controller/PC12: track 12.8 -> 63.0 mm
- net /Controller/PD11_SPI3_INT: track 0.00 -> 49.8 mm, vias 0 -> 4
- net /Controller/PC13: track 62.2 -> 12.8 mm
- net /Controller/PF9_USART6_TX: track 8.97 -> 57.1 mm, vias 2 -> 4
- net /Controller/PB0: track 46.0 -> 0.00 mm, vias 2 -> 0
- net GND: track 598.0 -> 626.7 mm, vias 901 -> 902
- net /Controller/PE3_TIM3_CH1: track 33.2 -> 48.2 mm
- net /Controller/PF1: track 33.2 -> 21.6 mm, vias 2 -> 3
- net /Controller/PD6_USART2_RX: track 0.00 -> 8.97 mm, vias 0 -> 2
- net +3V3: track 493.2 -> 497.5 mm
- net /Controller/PE13: track 57.3 -> 61.0 mm
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Other:
- board size 122 x 85 mm -> 142 x 85 mm
- board text added: "Trilithon Magi v2.1"
- board text added: "W"
- board text removed: "Trilithon Magi v2.0"
