File: Controller.kicad_sch (KiCad schematic)
At the start: 62 parts, among them J8 USB_C_Receptacle, J9 Conn_02x04, Q1 DMN32D2LFB4, SW1 SW_Push, U16 USB2514B, U17 CH390H, U18 STM32G0B1VETx, U19 TPD4EUSB30, Y2 25MHz, Y3 24MHz, Y4 32.768kHz

Commit message: Magi v2.1
Parts:
- removed R63: 2.49K, Resistor_SMD:R_0402_1005Metric, symbol Device:R
- added C190, C191: 100n, Capacitor_SMD:C_0402_1005Metric, symbol Device:C
- added R116, R117: 5.1k, Resistor_SMD:R_0402_1005Metric, symbol Device:R
- added TP13: TestPoint, TestPoint:TestPoint_Pad_D1.5mm, symbol Connector:TestPoint
- added U45: ATECC608B-MAHCZ, Package_DFN_QFN:DFN-8-1EP_3x2mm_P0.5mm_EP1.3x1.5mm, symbol Magi:ATECC608B-MAHCZ
- added U46: CAT25512HU5I-GT3, Magi:DFN-8-1EP_3x2mm_P0.5mm_EP0.9x1.4mm, symbol Memory_EEPROM:CAT250xxx-HU4
- D10, D7, D8, D9: value WS2812B -> WS2812C; footprint Magi:LED-SMD_4P-L4.0-W1.7-R -> Magi:LED-SMD_4P-L4.0-W1.7_DCS; LCSC C4154870 -> C55109523; MPN WS2812C-4020 -> WS2812C-4020-V6
Connections:
- net PB0 is gone; now on net PB0_MCU_BUTTON: U18.35 (PB0)
- net +3V3: now also C190.2, C191.2, R116.1, R117.1, U45.8 (VCC), U46.3 (~{WP}), U46.7 (~{HOLD}), U46.8 (VCC)
- net GND: now also C190.1, C191.1, U45.4 (GND), U45.9 (EP), U46.4 (GND), U46.9 (GND); no longer J9.5 (Pin_5)
- net PB3_SPI3_SCK: now also U46.6 (SCK)
- net PB4_SPI3_MISO: now also U46.2 (MISO)
- net PB5_SPI3_MOSI: now also U46.5 (MOSI)
- net PF1: now also R54.1, U16.26 (RESET_N)
- net PF9_USART6_TX: now also R116.2, TP13.1, U45.5 (SDA)
- net PC7: now reaches U18.58 (PC7)
- net PC7: now also R117.2, U46.1 (~{CS})
- net MCU_BUTTON renamed PB0_MCU_BUTTON
- net PB0_MCU_BUTTON: no longer U18.84 (PD6)
- net PD11 renamed PD11_SPI3_INT
- net PD11_SPI3_INT: now also J9.5 (Pin_5)
- new net PD6_USART2_RX: U18.84 (PD6)
- no-connect marks 28 -> 29
Other:
- moved on the sheet: C108, C109, C110, C111, C112, C113, C114, C115, C118, C123, C124, C125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
