File: EthernetSwitch.kicad_sch (KiCad schematic)
At the start: 53 parts, among them J7 RJ45_LED_Shielded, U13 RTL8367N, U14 TPD4EUSB30, U15 TPD4EUSB30, Y4 25MHz

Commit message: Magi v2.0
Parts:
- removed C101, C102, C103, C104, C105, C106, C107, C108, C111, C114, C115, C116: 100n, Capacitor_SMD:C_0402_1005Metric, symbol Device:C
- removed C109, C110: 6p, Capacitor_SMD:C_0402_1005Metric, symbol Device:C
- removed C112, C113: 100u, Capacitor_SMD:C_1206_3216Metric, symbol Device:C
- removed R51: 470R, Resistor_SMD:R_0402_1005Metric, symbol Device:R
- removed R52: 4.7k, Resistor_SMD:R_0402_1005Metric, symbol Device:R
- removed U13: RTL8367N, Magi:QFN-88_EP_10x10_Pitch0.4mm2, symbol Magi:RTL8367N
- added C67, C68, C69, C70, C71, C72, C75, C76, C77, C78, C81, C82, C83, C84, C85, C86, C87, C88, C89, C90: 100n, Capacitor_SMD:C_0402_1005Metric, symbol Device:C
- added C73, C74: 18pf, Capacitor_SMD:C_0402_1005Metric, symbol Device:C
- added C79: 10u, Capacitor_SMD:C_0603_1608Metric, symbol Device:C
- added C80: 1u, Capacitor_SMD:C_0402_1005Metric, symbol Device:C
- added L7: 2.2uH, Inductor_SMD:L_Changjiang_FTC404030S, symbol Device:L
- added U13: RTL8367S-CG, Package_QFP:LQFP-128_14x14mm_P0.4mm, symbol Magi:RTL8367S-CG
- C100: value 100u -> 100n; footprint Capacitor_SMD:C_1206_3216Metric -> Capacitor_SMD:C_0402_1005Metric; LCSC C15008 -> C307331; MPN CL31A107MQHNNNE -> CL05B104KB54PNC
- C95, C97, C98: value 100n -> 10u; footprint Capacitor_SMD:C_0402_1005Metric -> Capacitor_SMD:C_0603_1608Metric; LCSC C307331 -> C96446; MPN CL05B104KB54PNC -> CL10A106MA8NRNC
- C96: value 100n -> 1u; LCSC C307331 -> C29266; MPN CL05B104KB54PNC -> CL05A105KO5NNNC
- C99: value 100u -> 10u; footprint Capacitor_SMD:C_1206_3216Metric -> Capacitor_SMD:C_0603_1608Metric; LCSC C15008 -> C96446; MPN CL31A107MQHNNNE -> CL10A106MA8NRNC
- FB1, FB2: value FerriteBead -> 220R; footprint Inductor_SMD:L_1206_3216Metric -> Inductor_SMD:L_0603_1608Metric; LCSC C668306 -> C14709; MPN BLM31KN601SN1L -> BLM18PG121SN1D; Manufacturer Murata -> muRata
- J7: footprint Magi:RJ45-TH_MJ88B-B011-RVL11-P -> Magi:RJ45-TH_RJ45-005-202-11; LCSC C501462 -> C7421405; MPN MJ88B-B011-RVL11-P -> RJ45-005-202-11; Manufacturer Heling -> XUNPU
- R34: value 2.49K -> 5.1k; LCSC C852700 -> C25905; MPN RT0402BRD072K49L -> 0402WGF5101TCE; Manufacturer YAGEO -> Uniroyal
- R35, R36, R38, R39, R40: value 4.7k -> 5.1k; LCSC C25900 -> C25905; MPN 0402WGF4701TCE -> 0402WGF5101TCE
- R37: value 4.7k -> 2.49K; LCSC C25900 -> C25884; MPN 0402WGF4701TCE -> 0402WGF2491TCE
- R41, R42, R43, R44, R45, R47, R48, R49, R50: value 4.7k -> 1k; LCSC C25900 -> C11702; MPN 0402WGF4701TCE -> 0402WGF1001TCE
- R46: value 470R -> 1k; LCSC C25117 -> C11702; MPN 0402WGF4700TCE -> 0402WGF1001TCE
- TR1: value H2456G -> H2449G; footprint Magi:XFMR-SMD-24_L16.6-W9.0-LS9.6-BL -> Magi:RJ45-SMD_24P_L15.6-W8.7_H24308C; symbol Magi:H2456G -> Magi:H2449G; LCSC C5464750 -> C5464748; MPN H2456G -> H2449G
- U14, U15: footprint Magi:USON-10_2.5x1.0mm_P0.5mm -> Package_SON:USON-10_2.5x1.0mm_P0.5mm
- Y1: renamed from Y4; symbol Device:Crystal_GND24 -> Device:Crystal_GND24_Small; LCSC C127893 -> C20617996; MPN XRCGB25M000F3M00R0 -> XL7EL89COI-111YLC-25M; Manufacturer Murata -> YXC; private (none) -> KLC_S4.1
Connections:
- net ANALOG_1V1: now also C95.1, C96.1, C67.1, C68.1, C69.1, C70.1, C71.1, C72.1, C78.1, C81.1, U13.108 (AVDDL), U13.114 (PLLVDDL), U13.122 (AVDDL), U13.14 (AVDDL), U13.27 (AVDDL), U13.37 (SVDDL), U13.6 (AVDDL), U13.95 (AVDDL)
- net ANALOG_3V3: now also R34.2, C79.1, C80.1, C82.1, C83.1, C84.1, C85.1, C86.1, C87.1, C88.1, C89.1, C90.1, U13.102 (AVDDH), U13.11 (AVDDH), U13.116 (AVDDH), U13.128 (AVDDH), U13.17 (AVDDH), U13.21 (AVDDH), U13.33 (AVDDH), U13.41 (SVDDH), U13.82 (AVDDH), U13.90 (AVDDH); no longer C100.1, C92.1, C93.1, C94.1, C95.1, C96.1, C97.1, C98.1, R35.2
- net GND: now also R37.1, R38.2, R42.2, R44.2, R45.2, R46.2, C67.2, C68.2, C69.2, C70.2, C71.2, C72.2, C73.1, C74.1, C75.2, C76.2, C77.2, C78.2, C79.2, C80.2, C81.2, C82.2, C83.2, C84.2, C85.2, C86.2, C87.2, C88.2, C89.2, C90.2, U13.1 (GND), U13.105 (GND), U13.111 (GND), U13.115 (PLLGND), U13.119 (GND), U13.12 (AGND), U13.125 (GND), U13.18 (GND), U13.24 (GND), U13.32 (GND), U13.34 (SGND), U13.40 (SGND), U13.43 (GND), U13.44 (GND), U13.57 (GND), U13.61 (GND_SWR), U13.62 (GND_SWR), U13.68 (GND), U13.85 (GND), U13.89 (GND), U13.96 (GND), U13.99 (GND); no longer J7.9, R34.1, R36.2, R37.2, R39.2, R40.2, R49.2, R50.2
- net +3V3: now reaches R50.1
- net +3V3: now also C92.1, C93.1, C94.1, C97.1, C98.1, FB1.1, R35.2, R36.2, R39.2, R40.2, R41.2, R49.1, U13.42 (DVDDIO_2), U13.59 (DVDDIO_2), U13.65 (HV_SWR), U13.66 (HV_SWR), U13.67 (DVDDIO)
- net SMI_SCL: now reaches R36.1
- net SMI_SCL: now also U13.87 (SCK/GPIO54)
- net LAN0LED1: now reaches R39.1
- net LAN0LED1: now also J7.11, U13.80 (LED_DA/LAN0LED1/GPO51)
- net at R47.1: now also U13.55 (M2P_TXD2/M2M_RXD2/RG2_RXD2/GPIO11)
- net at R48.1: now also U13.56 (M2P_TXD3/M2M_RXD3/RG2_RXD3/GPIO12)
- net LAN0LED0: now reaches R40.1
- net LAN0LED0: now also J7.9, U13.81 (SMI_SEL/LED_CK/LAN0LED0/GPO52)
- net at R41.1: now also U13.60 (EN_SWR)
- net at R42.1: now also U13.50 (M2P_RXCLK/M2M_TXCLK/RG2_TXCLK/GPIO06)
- net at R43.1: now also U13.51 (M2P_TXCLK/M2M_RXCLK/RG2_RXCLK/GPIO07)
- net at Y1.3: now also C73.2, U13.84 (XTALI)
- net at Y1.1: now also C74.2, U13.83 (XTALO)
- net SMI_SDA: now reaches R35.1
- net SMI_SDA: now also U13.88 (SDA/GPIO55)
- net at J7.10: now also R50.2
- net at J7.12: now also R49.2; no longer R46.1
- net AUX_1V1 renamed 1V1
- net 1V1: now also C100.1, C99.1, C75.1, C76.1, C77.1, L7.2, U13.20 (DVDDL), U13.58 (DVDDL), U13.69 (DVDDL)
- removed net AUX_3V3: C99.1, FB1.1, R38.2, R41.2, R42.2, R44.2, R45.2, R46.2
- net ETH_SWITCH_SCK: no longer names the net of R45.1
- net ETH_SWITCH_SCK: now also U13.53 (SPIF_D1/M2P_TXD0/M2M_RXD0/RG2_RXD0/GPIO09)
- net ETH_SWITCH_SDA: no longer names the net of R38.1
- net ETH_SWITCH_SDA: now also U13.74 (EN_SPIF/LAN3LED0/GPO43)
- net P0LED0: no longer names the net of R44.1
- net P0LED0: now also U13.52 (M2P_TXEN/M2M_RXDV/RG2_RXCTL/GPIO08); no longer J7.11
- net P0MDIAN renamed MDIA-
- net MDIA-: now also TR1.3 (TD1-), U13.92 (P0MDIAN); no longer TR1.14 (TD4+)
- net P0MDIAP renamed MDIA+
- net MDIA+: now also TR1.2 (TD1+), U13.91 (P0MDIAP); no longer TR1.13 (TD4-)
- net P0MDIBN renamed MDIB-
- net MDIB-: now also TR1.6 (TD2-), U13.94 (P0MDIBN); no longer TR1.17
- net P0MDIBP renamed MDIB+
- net MDIB+: now also TR1.5 (TD2+), U13.93 (P0MDIBP); no longer TR1.16 (TD3-)
- net P0MDICN renamed MDIC-
- net MDIC-: now also TR1.9 (TD3-), U13.97 (P0MDICP); no longer TR1.20 (TD2+)
- net P0MDICP renamed MDIC+
- net MDIC+: now also TR1.8 (TD3+), U13.98 (P0MDICN); no longer TR1.19 (TD2-)
- net P0MDIDN renamed MDID-
- net MDID-: now also TR1.12 (TD4-), U13.101 (P0MDIDN); no longer TR1.23 (TD1+)
- net P0MDIDP renamed MDID+
- net MDID+: now also TR1.11 (TD4+), U13.100 (P0MDIDP); no longer TR1.22 (TD1-)
- net RJ47_DA_N renamed PORT_MDIA+
- net PORT_MDIA+: now also TR1.23 (MX1+); no longer TR1.11 (MX4+)
- net RJ47_DA_P renamed PORT_MDIA-
- net PORT_MDIA-: now also TR1.22 (MX1-); no longer TR1.12 (MX4-)
- net RJ47_DB_N renamed PORT_MDIB-
- net PORT_MDIB-: now also TR1.19 (MX2-); no longer TR1.8 (MX3+)
- net RJ47_DB_P renamed PORT_MDIB+
- net PORT_MDIB+: now also TR1.20 (MX2+); no longer TR1.9 (MX3-)
- net RJ47_DC_N renamed PORT_MDIC-
- net PORT_MDIC-: now also TR1.16 (MX3-); no longer TR1.5 (MX2+)
- net RJ47_DC_P renamed PORT_MDIC+
- net PORT_MDIC+: now also TR1.17 (MX3+); no longer TR1.6 (MX2-)
- net RJ47_DD_N renamed PORT_MDID-
- net PORT_MDID-: now also TR1.13 (MX4-); no longer TR1.2 (MX1+)
- net RJ47_DD_P renamed PORT_MDID+
- net PORT_MDID+: now also TR1.14 (MX4+); no longer TR1.3 (MX1-)
- new net: R37.2, U13.13 (MDIREF)
- new net: R46.1, U13.54 (SPIF_CS/M2P_TXD1/M2M_RXD1/RG2_RXD1/GPIO10)
- new net LX: L7.1, U13.63 (LX), U13.64 (LX)
- new net P1MDIA+: U13.103 (P1MDIAP)
- new net P1MDIA-: U13.104 (P1MDIAN)
- new net P1MDIB+: U13.106 (P1MDIBP)
- new net P1MDIB-: U13.107 (P1MDIBN)
- new net P1MDIC+: U13.109 (P1MDICP)
- new net P1MDIC-: U13.110 (P1MDICN)
- new net P1MDID+: U13.112 (P1MDIDP)
- new net P1MDID-: U13.113 (P1MDIDN)
- new net P2MDIA+: U13.117 (P2MDIAP)
- new net P2MDIA-: U13.118 (P2MDIAN)
- new net P2MDIB+: U13.120 (P2MDIBP)
- new net P2MDIB-: U13.121 (P2MDIBN)
- new net P2MDIC+: U13.123 (P2MDICP)
- new net P2MDIC-: U13.124 (P2MDICN)
- new net P2MDID+: U13.126 (P2MDIDP)
- new net P2MDID-: U13.127 (P2MDIDN)
- new net P3MDIA+: U13.2 (P3MDIAP)
- new net P3MDIA-: U13.3 (P3MDIAN)
- new net P3MDIB+: U13.4 (P3MDIBP)
- new net P3MDIB-: U13.5 (P3MDIBN)
- new net P3MDIC+: U13.7 (P3MDICP)
- new net P3MDIC-: U13.8 (P3MDICN)
- new net P3MDID+: U13.9 (P3MDIDP)
- new net P3MDID-: U13.10 (P3MDIDN)
- new net P4MDIA+: U13.22 (P4MDIAP)
- new net P4MDIA-: U13.23 (P4MDIAN)
- new net P4MDIB+: U13.25 (P4MDIBP)
- new net P4MDIB-: U13.26 (P4MDIBN)
- new net P4MDIC+: U13.28 (P4MDICP)
- new net P4MDIC-: U13.29 (P4MDICN)
- new net P4MDID+: U13.30 (P4MDIDP)
- new net P4MDID-: U13.31 (P4MDIDN)
- new net SGMII_RX+: U13.38 (HSIP)
- new net SGMII_RX-: U13.39 (HSIN)
- new net SGMII_TX+: U13.36 (HSOP)
- new net SGMII_TX-: U13.35 (HSON)
- new net ~{RESET}: R34.1, U13.86 (nRESET)
- no-connect marks 15 -> 25
Other:
- title: (none) -> Trilithon Magi
- moved on the sheet: FB2, J7, U14, U15
