File: Magi.kicad_sch (KiCad schematic)
At the start: 0 parts

Commit message: Magi v2.0
Parts:
- added H1, H2: MountingHole, Magi:MOUNTING-HOLE, symbol Mechanical:MountingHole_Pad
Connections:
- new net GND: H1.1, H2.1
- no-connect marks 0 -> 4
Other:
- sheet Control renamed Controller
- sheet Unit 1A renamed Unit 1
- sheet Unit 2A renamed Unit 2
- sheet Unit 3A renamed Unit 3
- removed sheet Unit 1B
- removed sheet Unit 2B
- removed sheet Unit 3B
- added sheet Interconnect (Connector.kicad_sch)
- added sheet USB (USB.kicad_sch)
- sheet Controller: file Control.kicad_sch -> Controller.kicad_sch
- sheet Controller ports: added ETH_P0+, ETH_P0-, ETH_P1+, ETH_P1-, HUB_USB2_1_D+, HUB_USB2_1_D-, HUB_USB2_2_D+, HUB_USB2_2_D-, HUB_USB2_3_D+, HUB_USB2_3_D-, PA1, PA15, PA2_LSCO, PA3, PA4_ADC1_IN4, PA5, PA6_I2C3_SDA, PA7_I2C3_SCL, PB0, PB1, PB10_ADC1_IN11, PB11_ADC1_IN15, PB12_ADC1_IN16, PB13_I2C2_SCL, PB14_I2C2_SDA, PB2_ADC1_IN10, PB6, PB7, PB8_I2C1_SCL, PB9_I2C1_SDA, PC1, PC10_USART4_TX, PC11_USART4_RX, PC12, PC13, PC4_USART1_TX, PC5_USART1_RX, PC6, PC8, PC9, PD10, PD11, PD12, PD13, PD14, PD15, PD4, PD5_USART2_TX, PD7, PD8_USART3_TX, PD9_USART3_RX, PE1, PE11, PE12, PE13, PE14, PE15, PE2, PE4, PE7, PE8, PE9, PF0, PF1, PF10, PF11, PF3, PF4, PF5, PF6, PF7, PF8, PF9_USART6_TX, UCPD1_CC1, UCPD1_CC2, UCPD2_CC1, UCPD2_CC2; removed none
- sheet Ethernet Switch ports: added P1MDIA+, P1MDIA-, P1MDIB+, P1MDIB-, P1MDIC+, P1MDIC-, P1MDID+, P1MDID-, P2MDIA+, P2MDIA-, P2MDIB+, P2MDIB-, P2MDIC+, P2MDIC-, P2MDID+, P2MDID-, P3MDIA+, P3MDIA-, P3MDIB+, P3MDIB-, P3MDIC+, P3MDIC-, P3MDID+, P3MDID-, P4MDIA+, P4MDIA-, P4MDIB+, P4MDIB-, P4MDIC+, P4MDIC-, P4MDID+, P4MDID-, SGMII_RX+, SGMII_RX-, SGMII_TX+, SGMII_TX-, SMI_SCL, SMI_SDA, ~{RESET}; removed none
- sheet Power ports: added CONN_5V_EN, CONN_DISCHARGE, CONN_VBUS_EN, ISENS_CONN_IN, ISENS_USB_IN, ISESN_CONN_OUT, USB_5V_EN, USB_DISCHARGE, VSENS_CONN, VSENS_USB; removed none
- sheet Unit 1: file Unit1A.kicad_sch -> Unit1.kicad_sch
- sheet Unit 1 ports: added 3V3_EN, 5V_EN, ACT_LED, CM_3V3, ETH_MDIA+, ETH_MDIA-, ETH_MDIB+, ETH_MDIB-, ETH_MDIC+, ETH_MDIC-, ETH_MDID+, ETH_MDID-, ID_SC, ID_SD, PWR_BTN, PWR_LED, RPIBOOT, RTC_CLOCK, UART_RX, UART_TX, USB2_D+, USB2_D-, ~{INTERRUPT}; removed none
- sheet Unit 2: file Unit2A.kicad_sch -> Unit2.kicad_sch
- sheet Unit 2 ports: added 3V3_EN, 5V_EN, ACT_LED, CM_3V3, ETH_MDIA+, ETH_MDIA-, ETH_MDIB+, ETH_MDIB-, ETH_MDIC+, ETH_MDIC-, ETH_MDID+, ETH_MDID-, ID_SC, ID_SD, PWR_BTN, PWR_LED, RPIBOOT, RTC_CLOCK, UART_RX, UART_TX, USB2_D+, USB2_D-, ~{INTERRUPT}; removed none
- sheet Unit 3: file Unit3A.kicad_sch -> Unit3.kicad_sch
- sheet Unit 3 ports: added 3V3_EN, 5V_EN, ACT_LED, CM_3V3, ETH_MDIA+, ETH_MDIA-, ETH_MDIB+, ETH_MDIB-, ETH_MDIC+, ETH_MDIC-, ETH_MDID+, ETH_MDID-, ID_SC, ID_SD, PWR_BTN, PWR_LED, RPIBOOT, RTC_CLOCK, UART_RX, UART_TX, USB2_D+, USB2_D-, USB3_0_D+, USB3_0_D-, USB3_0_RX+, USB3_0_RX-, USB3_0_TX+, USB3_0_TX-, USB3_1_D+, USB3_1_D-, USB3_1_RX+, USB3_1_RX-, USB3_1_TX+, USB3_1_TX-, ~{INTERRUPT}; removed none
- note removed: "Ethernet Switch"
- title: (none) -> Trilithon Magi

Commit message: Magi v2.1
Other:
- sheet Controller ports: added PD6_USART2_RX; removed PB0, PD11, PF1, PF9_USART6_TX
- sheet Unit 1 ports: added none; removed ~{INTERRUPT}
- sheet Unit 2 ports: added none; removed ~{INTERRUPT}
- sheet Unit 3 ports: added none; removed ~{INTERRUPT}
- moved on the sheet: H1, H2
