File: Power.kicad_sch (KiCad schematic)
At the start: 88 parts, among them J11 USB_C_Receptacle_USB2.0_16P, Q10 DMN32D2LFB4, Q11 DMN32D2LFB4, Q12 DMN32D2LFB4, Q13 DMN32D2LFB4, Q9 DMN32D2LFB4, U24 TVS2200DRV, U25 TPS259470A, U26 TPS259474A, U27 TPS62933, U28 TPS259470A, U29 CYPD3177-24LQ, U30 TPS62933

Commit message: Magi v2.0
Parts:
- removed BT1: RTC Battery, Magi:BAT-SMD_MY-1220-03, symbol Device:Battery_Cell
- removed C137: 47p C0G, Capacitor_SMD:C_0402_1005Metric, symbol Device:C
- removed C143: 1u 50V, Capacitor_SMD:C_0805_2012Metric, symbol Device:C
- removed C157, C158, C159, C168, C169, C170, C171, C172, C173, C174, C175, C176, C177, C178, C179, C180, C181, C182, C183, C184: 22u, Capacitor_SMD:C_0805_2012Metric, symbol Device:C
- removed C166: 100n, Capacitor_SMD:C_0402_1005Metric, symbol Device:C
- removed D4, D5: M7, Diode_SMD:D_SMA, symbol Device:D
- removed H1, H2: MountingHole, Magi:MOUNTING-HOLE, symbol Mechanical:MountingHole
- removed J11: USB_C_Receptacle_USB2.0_16P, Magi:USB-C-SMD_TYPEC-304J-BCP16, symbol Magi:USB_C_Receptacle_USB2.0_16P
- removed L7: 2.2u 4.5A, Inductor_SMD:L_Sunlord_MWSA0402S, symbol Device:L
- removed Q10, Q12, Q13, Q9: DMN32D2LFB4, Package_DFN_QFN:Diodes_DFN1006-3, symbol Device:Q_NMOS_GSD
- removed R69: 20k, Resistor_SMD:R_0402_1005Metric, symbol Device:R
- removed SYM1: Magi v1.0, Magi:NAMEPLATE, symbol Graphic:Logo_Open_Hardware_Small
- removed U24: TVS2200DRV, Package_SON:WSON-6-1EP_2x2mm_P0.65mm_EP1x1.6mm, symbol Power_Protection:TVS2200DRV
- removed U27, U30: TPS62933, Package_TO_SOT_SMD:SOT-583-8, symbol Regulator_Switching:TPS62933
- removed U29: CYPD3177-24LQ, Package_DFN_QFN:QFN-24-1EP_4x4mm_P0.5mm_EP2.75x2.75mm, symbol Interface_USB:CYPD3177-24LQ
- added C129, C134: 100n, Capacitor_SMD:C_0402_1005Metric, symbol Device:C
- added C130, C131, C135: 6.8n, Capacitor_SMD:C_0402_1005Metric, symbol Device:C
- added C144, C153: 22u, Capacitor_SMD:C_0805_2012Metric, symbol Device:C
- added C157, C158, C159: 100u, Capacitor_SMD:CP_Elec_6.3x5.7, symbol Device:C_Polarized
- added D11, D12: 4.3v, Diode_SMD:D_SOD-523, symbol Device:D_Zener
- added D13, D14, D15: RB161QS, Diode_SMD:D_SOD-882, symbol Device:D_Schottky
- added J10: Conn_02x02_Odd_Even, Connector_PinHeader_2.54mm:PinHeader_2x02_P2.54mm_Vertical, symbol Connector_Generic:Conn_02x02_Odd_Even
- added L9: 5.6uH, Inductor_SMD:L_Changjiang_FTC404030S, symbol Device:L
- added Q3, Q4: DMN32D2LFB4, Package_DFN_QFN:Diodes_DFN1006-3, symbol Device:Q_NMOS_GSD
- added R100, R89: 30R, Resistor_SMD:R_0402_1005Metric, symbol Device:R
- added R101, R93: 12k, Resistor_SMD:R_0402_1005Metric, symbol Device:R
- added R102, R95: 5.1k, Resistor_SMD:R_0402_1005Metric, symbol Device:R
- added R64, R65, R87, R99: 100k, Resistor_SMD:R_0402_1005Metric, symbol Device:R
- added R66, R92: 1.3k, Resistor_SMD:R_0402_1005Metric, symbol Device:R
- added R88: 37.4k, Resistor_SMD:R_0402_1005Metric, symbol Device:R
- added R94: 5.6k, Resistor_SMD:R_0402_1005Metric, symbol Device:R
- added R96: 1k, Resistor_SMD:R_0402_1005Metric, symbol Device:R
- added R97: 64.9k, Resistor_SMD:R_0402_1005Metric, symbol Device:R
- added R98: 1.2k 0.5W, Resistor_SMD:R_1206_3216Metric, symbol Device:R
- added TP10, TP11, TP12, TP13, TP8, TP9: TestPoint, TestPoint:TestPoint_Pad_D1.5mm, symbol Connector:TestPoint
- added U20, U21, U23, U24: TPS259470A, Magi:RPW0010A-MFG, symbol Magi:TPS259470ARPWR
- added U26, U28: TPS56339DDC, Package_TO_SOT_SMD:SOT-23-6, symbol Regulator_Switching:TPS56339DDC
- C132: renamed from C135; footprint Capacitor_SMD:C_0603_1608Metric -> Capacitor_SMD:C_0402_1005Metric; LCSC C162241 -> C1518206; MPN GRM1885C1H682JA01D -> GRM1555C1H682JE01D; Manufacturer Murata -> muRata
- C133: renamed from C134; value 3.3u 100V -> 10u 50V; LCSC C575409 -> C126612; MPN C3225X7S2A335KT000N -> GCM32EC71H106KA03L; Manufacturer TDK -> muRata
- C136: value 100n -> 6.8n; LCSC C307331 -> C1518206; MPN CL05B104KB54PNC -> GRM1555C1H682JE01D; Manufacturer Samsung -> muRata
- C137: renamed from C144; footprint Capacitor_SMD:C_0603_1608Metric -> Capacitor_SMD:C_0402_1005Metric; LCSC C162241 -> C1518206; MPN GRM1885C1H682JA01D -> GRM1555C1H682JE01D; Manufacturer Murata -> muRata
- C138, C148: value 10u 50V -> 22u; LCSC C15850 -> C45783; MPN CL21A106KAYNNNE -> CL21A226MAQNNNE
- C139: value 100n 50V -> 100n
- C140: value 1u 50V -> 100n; footprint Capacitor_SMD:C_0805_2012Metric -> Capacitor_SMD:C_0402_1005Metric; LCSC C28323 -> C307331; MPN CL21B105KBFNNNE -> CL05B104KB54PNC
- C141, C142, C147: value 100n -> 22u; footprint Capacitor_SMD:C_0402_1005Metric -> Capacitor_SMD:C_0805_2012Metric; LCSC C307331 -> C45783; MPN CL05B104KB54PNC -> CL21A226MAQNNNE
- C143: renamed from C153; footprint Capacitor_SMD:C_0603_1608Metric -> Capacitor_SMD:C_0402_1005Metric; LCSC C162241 -> C1518206; MPN GRM1885C1H682JA01D -> GRM1555C1H682JE01D; Manufacturer Murata -> muRata
- C145: value 22u -> 100n; footprint Capacitor_SMD:C_0805_2012Metric -> Capacitor_SMD:C_0402_1005Metric; LCSC C45783 -> C307331; MPN CL21A226MAQNNNE -> CL05B104KB54PNC
- C146: value 33n -> 100n; footprint Capacitor_SMD:C_0603_1608Metric -> Capacitor_SMD:C_0402_1005Metric; LCSC C21117 -> C307331; MPN CL10B333KB8NNNC -> CL05B104KB54PNC
- C149: value 100n 50V -> 22u; footprint Capacitor_SMD:C_0402_1005Metric -> Capacitor_SMD:C_0805_2012Metric; LCSC C307331 -> C45783; MPN CL05B104KB54PNC -> CL21A226MAQNNNE
- C150, C151: value 100u -> 22u; footprint Capacitor_SMD:C_1206_3216Metric -> Capacitor_SMD:C_0805_2012Metric; LCSC C15008 -> C45783; MPN CL31A107MQHNNNE -> CL21A226MAQNNNE
- C152: value 33n -> 22u; footprint Capacitor_SMD:C_0603_1608Metric -> Capacitor_SMD:C_0805_2012Metric; LCSC C21117 -> C45783; MPN CL10B333KB8NNNC -> CL21A226MAQNNNE
- L8: value 2.2u 4.5A -> 4.7uH; footprint Inductor_SMD:L_Sunlord_MWSA0402S -> Inductor_SMD:L_Changjiang_FTC404030S; LCSC C408335 -> C39676083; MPN MWSA0402S-2R2MT -> FTC404030S4R7MGCA; Manufacturer Sunlord -> cjiang
- R67: value 220k 1% -> 5.6k; LCSC C25767 -> C409920; MPN 0402WGF2203TCE -> RC0402FR-075K6L; Manufacturer Uniroyal -> Panasonic
- R68, R80: value 100k -> 1.3k; LCSC C25741 -> C25866; MPN 0402WGF1003TCE -> 0402WGF1301TCE
- R69: renamed from R66; value 100k -> 12k; LCSC C25741 -> C25752; MPN 0402WGF1003TCE -> 0402WGF1202TCE
- R70: value 2.26k 1% -> 5.1k; LCSC C208833 -> C25905; MPN RMS04FT2261 -> 0402WGF5101TCE; Manufacturer TA-I Tech -> Uniroyal
- R71: value 953 -> 5.1k; LCSC C227278 -> C25905; MPN AC0402FR-07953RL -> 0402WGF5101TCE; Manufacturer YAGEO -> Uniroyal
- R72: value 13k 1% -> 5.6k; LCSC C138057 -> C409920; MPN RC0402FR-0713KL -> RC0402FR-075K6L; Manufacturer YAGEO -> Panasonic
- R73: value 30.9k 1% -> 100k; LCSC C416514 -> C25741; MPN ERJ2RKF3092X -> 0402WGF1003TCE; Manufacturer PANASONIC -> Uniroyal
- R74: value 953 -> 1k; LCSC C227278 -> C11702; MPN AC0402FR-07953RL -> 0402WGF1001TCE; Manufacturer YAGEO -> Uniroyal
- R75, R85: value 10k 1% -> 1k; LCSC C25744 -> C11702; MPN 0402WGF1002TCE -> 0402WGF1001TCE
- R76: value 15k -> 1k; footprint Capacitor_SMD:C_0402_1005Metric -> Resistor_SMD:R_0402_1005Metric; LCSC C25756 -> C11702; MPN 0402WGF1502TCE -> 0402WGF1001TCE
- R77: value 220k 1% -> 100k; LCSC C25767 -> C25741; MPN 0402WGF2203TCE -> 0402WGF1003TCE
- R79: value 2.74k 1% -> 5.6k; LCSC C705693 -> C409920; MPN RT0402FRE072K74L -> RC0402FR-075K6L; Manufacturer YAGEO -> Panasonic
- R81: value 2.4k -> 5.1k; LCSC C25882 -> C25905; MPN 0402WGF2401TCE -> 0402WGF5101TCE
- R82: value 20k -> 5.1k; LCSC C25765 -> C25905; MPN 0402WGF2002TCE -> 0402WGF5101TCE
- R83: value 12.7k 1% -> 100k; LCSC C138059 -> C25741; MPN RC0402FR-0712K7L -> 0402WGF1003TCE; Manufacturer YAGEO -> Uniroyal
- R84: value 3.74k 1% -> 1k; LCSC C137989 -> C11702; MPN RC0402FR-073K74L -> 0402WGF1001TCE; Manufacturer YAGEO -> Uniroyal
- R86: value 1.2k 1% -> 1k; LCSC C144793 -> C11702; MPN AC0402FR-071K2L -> 0402WGF1001TCE; Manufacturer YAGEO -> Uniroyal
- R90: value 5.1k -> 1.2k 0.5W; footprint Resistor_SMD:R_0402_1005Metric -> Resistor_SMD:R_1206_3216Metric; LCSC C25905 -> C7468365; MPN 0402WGF5101TCE -> FRP1206F1201TS; Manufacturer Uniroyal -> FOJAN
- R91: value 1k -> 100k; LCSC C11702 -> C25741; MPN 0402WGF1001TCE -> 0402WGF1003TCE
- U25: renamed from U26; value TPS259474A -> TPS259470A; LCSC C3662807 -> C3662799; MPN TPS259474ARPWR -> TPS259470ARPWR
- renumbered Q11 to Q2, U25 to U22, U28 to U27
Connections:
- net +20V: now also C149.1, C150.1, C151.1, C152.1, C153.1, C157.1, C158.1, C159.1, D13.1 (K), J10.1 (Pin_1), J10.3 (Pin_3), TP10.1
- net GND: now also C133.2, C136.2, C138.1, C139.1, C141.2, C142.2, C145.1, C147.2, R67.1, R70.1, R71.1, R78.1, R79.1, R84.2, C129.2, C130.2, C131.2, C134.2, C135.2, C144.1, C153.2, C157.2, C158.2, C159.2, D11.2 (A), D12.2 (A), D13.2 (A), D14.2 (A), D15.2 (A), J10.2 (Pin_2), J10.4 (Pin_4), Q3.2 (S), Q4.2 (S), R101.2, R102.1, R93.2, R94.2, R95.1, R96.2, TP12.1, TP13.1, U20.8 (GND), U21.8 (GND), U23.8 (GND), U24.8 (GND), U26.1 (GND), U28.1 (GND); no longer C133.1, C138.2, C139.2, C140.1, C141.1, C142.1, C145.2, C146.2, R71.2, R83.2, R91.2
- net ISENS_CONN_IN: now also R96.1; no longer R86.1
- net ISENS_USB_IN: now also R76.1; no longer R71.1
- net PWR_MUX: now also C138.2, C139.2, C145.2, C144.2, TP11.1, U21.6 (OUT), U24.6 (OUT), U26.3 (VIN), U28.3 (VIN); no longer C138.1, C139.1, C148.1, C149.1
- net VBUS: now also R73.1, R90.1, R91.1, D15.1 (K), R64.1, R65.1, TP8.1, U20.6 (OUT), U21.5 (IN); no longer C133.2, R67.1, R68.2
- net at R85.1: now also U24.9 (ILM); no longer R84.2
- net at R73.2: now also C129.1, D11.1 (K), U21.1 (EN/UVLO); no longer R75.1
- net at R80.1: now also R77.2; no longer R82.2
- net at R68.1: now also R65.2
- net +5V: now reaches C147.1
- net +5V: now also C148.1, L9.2, R97.1, U20.5 (IN), U23.5 (IN); no longer L8.1
- net CONN_5V_EN: now reaches R81.2
- net CONN_5V_EN: now also U23.1 (EN/UVLO); no longer R78.1
- net at C136.1: now also U24.7 (dVdt)
- net at Q2.2 (S), U27.2 (OVLO): now also R92.2, R94.1; no longer R79.2, R83.1
- net BUCK_SW_5: now reaches C146.1
- net BUCK_SW_5: now also L9.1, U28.2 (SW)
- net at C140.2: now also R89.2
- removed net AUX_1V1: C150.1, C151.1, L8.2, R84.1
- removed net AUX_3V3: C145.1, R69.2, R73.1
- net CONN_VBUS renamed VCON
- net VCON: now also C133.1, R83.1, D14.1 (K), R87.1, R98.1, R99.1, TP9.1, U23.6 (OUT), U24.5 (IN); no longer R80.2
- removed net CYPD3177_VDDD: C141.2, C142.2, R78.2, R90.2
- net ISENS_CONN_OUT: no longer names the net of R74.1
- net ISENS_CONN_OUT: now also U20.9 (ILM); no longer U25.9 (ILM)
- net USB_OVLO renamed VBUS_OVLO
- net VBUS_OVLO: now also R66.2; no longer R70.2
- removed net USB_UVLO: R67.2, R70.1, U22.1 (EN/UVLO), U25.1 (EN/UVLO)
- new net: R84.1, U23.9 (ILM)
- new net: R64.2, R66.1, U22.1 (EN/UVLO)
- new net: Q3.3 (D), R90.2
- new net: R67.2, R68.2, U21.2 (OVLO)
- new net: R100.1, U28.6 (BOOT)
- new net: C146.2, R100.2
- new net: R101.1, R97.2, U28.4 (FB)
- new net: R88.2, R93.1, U26.4 (FB)
- new net: Q4.3 (D), R98.2
- new net: C130.1, U20.7 (dVdt)
- new net: R87.2, R92.1, U27.1 (EN/UVLO)
- new net: C134.1, D12.1 (K), R83.2, U24.1 (EN/UVLO)
- new net: C131.1, U21.7 (dVdt)
- new net: R75.1, U21.9 (ILM)
- new net: C135.1, U23.7 (dVdt)
- new net: R82.2, U23.2 (OVLO)
- new net: R71.2, U20.2 (OVLO)
- new net: R79.2, R80.2, U24.2 (OVLO)
- new net: R89.1, U26.6 (BOOT)
- new net +3V3: C141.1, C142.1, L8.2, R69.2, R88.1
- new net BUCK_SW_3: C140.1, L8.1, U26.2 (SW)
- new net CONN_DISCHARGE: Q4.1 (G)
- new net CONN_VBUS_EN: R78.2, U25.1 (EN/UVLO)
- new net ISESN_CONN_OUT: R86.1, U25.9 (ILM)
- new net USB_5V_EN: R70.2, U20.1 (EN/UVLO)
- new net USB_DISCHARGE: Q3.1 (G)
- new net VSENS_CONN: R102.2, R99.2
- new net VSENS_USB: R91.2, R95.2
- no-connect marks 25 -> 21
Other:
- note added: "UVLO: 18.59V = 1.2*(100+1.3+5.6)/(1.3+5.6) OVLO: 22.91V = 1.2*(100+1.3+5.6)/5.6"
- note removed: "1.1V @ 1.5A"
- note removed: "3.3V @ 1.5A"
- note removed: "RTC battery"
- note removed: "USB PD"
- title: (none) -> Trilithon Magi
- moved on the sheet: C132, C133, C137, C143, Q2, R69, U22, U25, U27

Commit message: Magi v2.1
Parts:
- added TP12, TP16: TestPoint, TestPoint:TestPoint_Pad_D1.5mm, symbol Connector:TestPoint
- renumbered TP12 to TP14, TP13 to TP15
Connections:
- net +3V3: now also TP12.1
- net GND: now also TP16.1
Other:
- moved on the sheet: J10, TP14, TP15
