File: Unit1.kicad_sch (KiCad schematic)
At the start: 45 parts, among them J1 Micro_SD_Card_Det2, J2 Bus_M.2_Socket_M, U1 TPS56339DDC, U2 TPS56339DDC, U3 AP2151W, U4 74AUP1G125

Commit message: Magi v2.1
Connections:
- net ~{INTERRUPT}: no longer names the net of Module1.24 (GPIO26)
- no-connect marks 30 -> 31
Changed lines of the file:
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@@
 	(title_block
 		(title "Trilithon Magi")
-		(rev "2.0")
+		(date "2026-10-06")
+		(rev "2.1")
 	)
 	(rectangle
@@
 	)
 	(no_connect
+		(at 34.29 72.39)
+	)
+	(no_connect
 		(at 97.79 132.08)
 	)
@@
 		)
 	)
-	(hierarchical_label "~{INTERRUPT}"
-		(shape input)
-		(at 34.29 72.39 180)
-		(effects
-			(font
-				(size 1.27 1.27)
-			)
-			(justify right)
-		)
-	)
