File: Unit2.kicad_sch (KiCad schematic)
At the start: 45 parts, among them J3 Micro_SD_Card_Det2, J4 Bus_M.2_Socket_M, U5 TPS56339DDC, U6 TPS56339DDC, U7 AP2151W, U8 74AUP1G125

Commit message: Magi v2.1
Connections:
- net ~{INTERRUPT}: no longer names the net of Module2.24 (GPIO26)
- no-connect marks 30 -> 31
Changed lines of the file:
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@@
 	(title_block
 		(title "Trilithon Magi")
-		(rev "2.0")
+		(date "2026-10-06")
+		(rev "2.1")
 	)
 	(rectangle
@@
 	)
 	(no_connect
+		(at 34.29 73.66)
+	)
+	(no_connect
 		(at 99.06 125.73)
 	)
@@
 		(effects
 			(font
-				(size 1.27 1.27)
-			)
-			(justify right)
-		)
-	)
-	(hierarchical_label "~{INTERRUPT}"
-		(shape input)
-		(at 34.29 73.66 180)
-		(effects
-			(font
