File: Unit3.kicad_sch (KiCad schematic)
At the start: 45 parts, among them J5 Micro_SD_Card_Det2, J6 Bus_M.2_Socket_M, U10 TPS56339DDC, U11 AP2151W, U12 74AUP1G125, U9 TPS56339DDC

Commit message: Magi v2.1
Connections:
- net ~{INTERRUPT}: no longer names the net of Module3.24 (GPIO26)
- no-connect marks 18 -> 19
Changed lines of the file:
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@@
 	(title_block
 		(title "Trilithon Magi")
-		(rev "2.0")
+		(date "2026-10-06")
+		(rev "2.1")
 	)
 	(rectangle
@@
 	)
 	(no_connect
+		(at 35.56 77.47)
+	)
+	(no_connect
 		(at 129.54 99.06)
 	)
@@
 		)
 	)
-	(hierarchical_label "~{INTERRUPT}"
-		(shape input)
-		(at 35.56 77.47 180)
-		(effects
-			(font
-				(size 1.27 1.27)
-			)
-			(justify right)
-		)
-	)
